File: 1_PCB/PowerMonitor.kicad_pcb (KiCad board)
At the start: 4 copper layers, 50 x 44.5 mm, 68 parts, among them J1 Conn_01x07, J2 Conn_01x02, J3 Conn_01x02, J4 Conn_01x02, J5 Conn_01x02, J6 Conn_01x02, J8 Conn_01x02, J9 Conn_01x02, Q1 STL325N4LF8AG, U1 BQ76942, U2 STM32G031K8Ux, U3 BD9E302EFJ, U4 BD9E302EFJ

Commit message: DEBUG: Fixed circuit bugs - Added I2C pull-up resistors - Fixed BQ76942 REG pin bugs - Added temperature sensor
Parts:
- added C11: 0.1uF, Capacitor_SMD:C_0402_1005Metric, F.Cu at (159.8, 113.9)
- added C13: 0.47uF, Capacitor_SMD:C_0402_1005Metric, F.Cu at (148.9, 112.6)
- added R28: 10k, Resistor_SMD:R_0402_1005Metric, F.Cu at (146.9, 109.8)
- added R29: 10k, Resistor_SMD:R_0402_1005Metric, F.Cu at (145.9, 109.8)
- added TP4: TestPoint, TestPoint:TestPoint_Pad_D1.0mm, F.Cu at (148.8, 110.5)
- added TP5: TestPoint, TestPoint:TestPoint_Pad_D1.0mm, F.Cu at (143.8, 109.3)
- moved TP3 1.13 mm to (161.3, 114.4)
- moved R11 0.30 mm to (150.2, 114.5)
- moved R10 0.25 mm to (151.2, 114.5)
Connections:
- U1 pad 21: unconnected-(U1-TS1-Pad21) -> Temp
- U1 pad 22: unconnected-(U1-TS2-Pad22) -> BAT_BALANCE_0
- U1 pad 24: unconnected-(U1-REG18-Pad24) -> Net-(U1-REG18)
- U1 pad 36: unconnected-(U1-REGIN-Pad36) -> BAT_BALANCE_0
- U1 pad 37: unconnected-(U1-BREG-Pad37) -> BAT_BALANCE_0
Routing:
- net +3.3V: track 28.9 -> 49.0 mm, vias 1 -> 2
- net BAT_BALANCE_0: track 141.2 -> 159.3 mm, vias 63 -> 64
- net OUT-: track 124.5 -> 131.9 mm, vias 67 -> 69
- net Temp: track 0.00 -> 6.21 mm
- net SDA: track 21.4 -> 24.1 mm
- net Net-(U1-REG18): track 0.00 -> 1.05 mm
- net Net-(U1-DSG): track 28.7 -> 27.7 mm, vias 2 -> 3
- net ARM_SW: track 31.2 -> 32.1 mm
- net NRST: track 2.07 -> 2.81 mm
Other:
- board text added: "2026.07.20"
- board text added: "TEMP+"
- board text added: "TEMP-"
- board text removed: "2026.04.02"
